File: 555-pwm-motor driver/kicad files/555-pwm-motor driver.kicad_sch (KiCad schematic)
At the start: 17 parts, among them J1 Screw_Terminal_01x02, J2 Screw_Terminal_01x02, Q1 IRLZ44N, U1 LM7805_TO220, U2 SE555P, U3 3PIN-POT-LOCAL

Commit message: Adding pcb files-closes #1
Parts:
- added J3, J4: Conn_01x01_Male, Connector_PinHeader_1.00mm:PinHeader_1x01_P1.00mm_Vertical, symbol Connector:Conn_01x01_Male
Connections:
- net at C4.1, U2.6 (THR), U3.2 (VR): now also J4.1 (Pin_1); no longer U2.2 (TR)
- new net: J3.1 (Pin_1), U2.2 (TR)
Changed lines of the file:
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@@
 (kicad_sch (version 20211123) (generator eeschema)
   (paper "A4")
+  (junction (at 162.56 101.6) (diameter 0) (color 0 0 0 0)
+  )
   (junction (at 83.82 85.09) (diameter 0) (color 0 0 0 0)
   )
   (junction (at 52.07 85.09) (diameter 0) (color 0 0 0 0)
   )
-  (junction (at 162.56 101.6) (diameter 0) (color 0 0 0 0)
-  )
   (junction (at 171.45 88.9) (diameter 0) (color 0 0 0 0)
   )
@@
     (stroke (width 0) (type default) (color 0 0 0 0))
   )
-  (wire (pts (xy 162.56 114.3) (xy 162.56 101.6))
-    (stroke (width 0) (type default) (color 0 0 0 0))
-  )
   (wire (pts (xy 83.82 97.79) (xy 88.9 97.79))
     (stroke (width 0) (type default) (color 0 0 0 0))
@@
     (stroke (width 0) (type default) (color 0 0 0 0))
   )
+  (wire (pts (xy 170.18 105.41) (xy 162.56 105.41))
+    (stroke (width 0) (type default) (color 0 0 0 0))
+  )
   (wire (pts (xy 214.63 81.28) (xy 220.98 81.28))
     (stroke (width 0) (type default) (color 0 0 0 0))
@@
     (stroke (width 0) (type default) (color 0 0 0 0))
   )
+  (wire (pts (xy 83.82 85.09) (xy 88.9 85.09))
+    (stroke (width 0) (type default) (color 0 0 0 0))
+  )
   (wire (pts (xy 60.96 72.39) (xy 64.77 72.39))
     (stroke (width 0) (type default) (color 0 0 0 0))
@@
     (stroke (width 0) (type default) (color 0 0 0 0))
   )
-  (wire (pts (xy 106.68 86.36) (xy 106.68 114.3))
-    (stroke (width 0) (type default) (color 0 0 0 0))
-  )
   (wire (pts (xy 171.45 100.33) (xy 189.23 100.33))
     (stroke (width 0) (type default) (color 0 0 0 0))
@@
     (stroke (width 0) (type default) (color 0 0 0 0))
   )
-  (wire (pts (xy 83.82 85.09) (xy 88.9 85.09))
-    (stroke (width 0) (type default) (color 0 0 0 0))
-  )
   (wire (pts (xy 162.56 91.44) (xy 162.56 88.9))
     (stroke (width 0) (type default) (color 0 0 0 0))
@@
     (stroke (width 0) (type default) (color 0 0 0 0))
   )
-  (wire (pts (xy 106.68 114.3) (xy 162.56 114.3))
-    (stroke (width 0) (type default) (color 0 0 0 0))
-  )
   (wire (pts (xy 162.56 86.36) (xy 165.1 86.36))
     (stroke (width 0) (type default) (color 0 0 0 0))
@@
     (stroke (width 0) (type default) (color 0 0 0 0))
   )
+  (wire (pts (xy 106.68 81.28) (xy 106.68 86.36))
+    (stroke (width 0) (type default) (color 0 0 0 0))
+  )
   (wire (pts (xy 149.86 77.47) (xy 149.86 81.28))
     (stroke (width 0) (type default) (color 0 0 0 0))
@@
     (stroke (width 0) (type default) (color 0 0 0 0))
   )
+  (wire (pts (xy 162.56 105.41) (xy 162.56 101.6))
+    (stroke (width 0) (type default) (color 0 0 0 0))
+  )
   (wire (pts (xy 189.23 87.63) (xy 196.85 87.63))
     (stroke (width 0) (type default) (color 0 0 0 0))
   )
   (wire (pts (xy 186.69 78.74) (xy 186.69 88.9))
+    (stroke (width 0) (type default) (color 0 0 0 0))
+  )
+  (wire (pts (xy 120.65 81.28) (xy 106.68 81.28))
     (stroke (width 0) (type default) (color 0 0 0 0))
   )
@@
     (pin "2")
   )
+  (symbol (lib_id "Connector:Conn_01x01_Male") (at 115.57 81.28 0) (unit 1)
+    (in_bom yes) (on_board yes) (fields_autoplaced)
+    (property "Reference" "J3" (id 0) (at 116.205 76.2 0))
+    (property "Value" "Conn_01x01_Male" (id 1) (at 116.205 78.74 0))
+    (property "Footprint" "Connector_PinHeader_1.00mm:PinHeader_1x01_P1.00mm_Vertical" (id 2) (at 115.57 81.28 0)
+      (effects (font (size 1.27 1.27)) hide)
+    )
+    (property "Datasheet" "~" (id 3) (at 115.57 81.28 0)
+      (effects (font (size 1.27 1.27)) hide)
+    )
+    (pin "1")
+  )
   (symbol (lib_id "Device:LED") (at 57.15 72.39 0) (unit 1)
     (in_bom yes) (on_board yes) (fields_autoplaced)
@@
     (pin "2")
   )
+  (symbol (lib_id "Connector:Conn_01x01_Male") (at 165.1 105.41 0) (unit 1)
+    (in_bom yes) (on_board yes)
+    (property "Reference" "J4" (id 0) (at 165.735 100.33 0))
+    (property "Value" "Conn_01x01_Male" (id 1) (at 165.1 107.95 0))
+    (property "Footprint" "Connector_PinHeader_1.00mm:PinHeader_1x01_P1.00mm_Vertical" (id 2) (at 165.1 105.41 0)
+      (effects (font (size 1.27 1.27)) hide)
+    )
+    (property "Datasheet" "~" (id 3) (at 165.1 105.41 0)
+      (effects (font (size 1.27 1.27)) hide)
+    )
+    (pin "1")
+  )
   (sheet_instances
     (path "/" (page "1"))
@@
       (reference "J2") (unit 1) (value "Screw_Terminal_01x02") (footprint "TerminalBlock_Phoenix:TerminalBlock_Phoenix_MKDS-1,5-2-5.08_1x02_P5.08mm_Horizontal")
     )
+    (path "/97323fc5-de14-4640-a522-92e44133a8b5"
+      (reference "J3") (unit 1) (value "Conn_01x01_Male") (footprint "Connector_PinHeader_1.00mm:PinHeader_1x01_P1.00mm_Vertical")
+    )
+    (path "/e9ab0d29-4a38-4efd-8bdd-680c70670e7d"
+      (reference "J4") (unit 1) (value "Conn_01x01_Male") (footprint "Connector_PinHeader_1.00mm:PinHeader_1x01_P1.00mm_Vertical")
+    )
     (path "/459987b2-019a-437e-9e72-46657e461bc8"
